Commit message: Basic wind force plugin setup
A basic setup is completed with force being acted on the quad simulating
the action of wind in a direction

File: iarc_simulation_tools/urdf/gazebo_wind_plugin.xacro (robot description, xacro)
@@ -1,9 +1,11 @@
 <?xml version="1.0"?>
 <robot xmlns:xacro="http://ros.org/wiki/xacro">
-  <xacro:macro name="gazebo_wind_plugin_macro" params="namespace">
+  <xacro:macro name="gazebo_wind_plugin_macro" params="namespace link_name windspeed windangle">
     <gazebo>
       <plugin name="wind_plugin" filename="libiarc_wind_plugin.so">
         <namespace>${namespace}</namespace>
-        <linkName>${namespace}/base_link</linkName>
+        <link_name>${namespace}/base_link</link_name>
+        <windspeed>${windspeed}</windspeed>
+        <windangle>${windangle}</windangle>
       </plugin>
     </gazebo>

File: iarc_simulation_tools/urdf/mav.xacro (robot description, xacro)
@@ -51,5 +51,8 @@
   </xacro:rgbd_sensor_depth_macro>
   <xacro:gazebo_wind_plugin_macro
-    namespace="${namespace}"  >
+    namespace="${namespace}"
+    link_name="${namespace}/base_link"
+    windspeed = "5"
+    windangle = "0"  >
   </xacro:gazebo_wind_plugin_macro>
 </robot>

Commit message: Clean code and add precision generality
Minor changes in code formatting and modified the code block
responsible for calculating floor and ceil of the input value to make
it general. Added precision as a sdf parameter.

File: iarc_simulation_tools/urdf/gazebo_wind_plugin.xacro (robot description, xacro)
@@ -1,5 +1,5 @@
 <?xml version="1.0"?>
 <robot xmlns:xacro="http://ros.org/wiki/xacro">
-  <xacro:macro name="gazebo_wind_plugin_macro" params="namespace link_name windspeed windangle">
+  <xacro:macro name="gazebo_wind_plugin_macro" params="namespace link_name windspeed windangle precision">
     <gazebo>
       <plugin name="wind_plugin" filename="libiarc_wind_plugin.so">
@@ -8,4 +8,5 @@
         <windspeed>${windspeed}</windspeed>
         <windangle>${windangle}</windangle>
+        <precision>${precision}</precision>
       </plugin>
     </gazebo>

File: iarc_simulation_tools/urdf/mav.xacro (robot description, xacro)
@@ -53,6 +53,7 @@
     namespace="${namespace}"
     link_name="${namespace}/base_link"
-    windspeed = "5"
-    windangle = "0"  >
+    windspeed = "2"
+    windangle = "1.57"
+    precision = "0.5"  >
   </xacro:gazebo_wind_plugin_macro>
 </robot>
