Commit message: Add camera to quadrotor

File: iarc_simulation_tools/urdf/quadrotor.xacro (robot description, xacro)
@@ -130,3 +130,15 @@
     <xacro:insert_block name="rotor_inertia" />
   </xacro:vertical_rotor>
+  <xacro:rgbd_sensor_depth_macro
+  namespace="${namespace}" parent_link="${namespace}/base_link"
+  camera_suffix="depth"
+  frame_rate="30.0"
+  fov = "1.59174"
+  baseline = "0.05"
+  width = "848"
+  height = "480"
+  max_range="50.0"
+  min_range="0.195">
+  <origin xyz="0.0 -0.2 -0.05" rpy="0 0.1 -1.57" />
+</xacro:rgbd_sensor_depth_macro>
 </robot>

File: iarc_simulation_tools/urdf/quadrotor_base.xacro (robot description, xacro)
@@ -3,4 +3,5 @@
   <xacro:include filename="$(find rotors_description)/urdf/component_snippets.xacro" />
   <!-- Instantiate iris "mechanics" -->
+  <xacro:include filename="$(find iarc_simulation_tools)/urdf/rgbd_camera.xacro"/>
   <xacro:include filename="$(find iarc_simulation_tools)/urdf/quadrotor.xacro" />
   <!-- Instantiate a controller. -->

Commit message: Align quadrotor hooks in proper direction

File: iarc_simulation_tools/urdf/quadrotor.xacro (robot description, xacro)
@@ -5,5 +5,5 @@
   <xacro:property name="rotor_velocity_slowdown_sim" value="10" />
   <xacro:property name="use_mesh_file" value="true" />
-  <xacro:property name="mesh_file" value="package://iarc_simulation_tools/models/quadrotor/meshes/quadrotor.dae" />
+  <xacro:property name="mesh_file" value="package://iarc_simulation_tools/models/quadrotor/meshes/quadrotor_2.dae" />
   <xacro:property name="mass" value="1.5" /> <!-- [kg] -->
   <xacro:property name="body_width" value="0.47" /> <!-- [m] -->
@@ -131,14 +131,14 @@
   </xacro:vertical_rotor>
   <xacro:rgbd_sensor_depth_macro
-  namespace="${namespace}" parent_link="${namespace}/base_link"
-  camera_suffix="depth"
-  frame_rate="30.0"
-  fov = "1.59174"
-  baseline = "0.05"
-  width = "848"
-  height = "480"
-  max_range="50.0"
-  min_range="0.195">
-  <origin xyz="0.0 -0.2 -0.05" rpy="0 0.1 -1.57" />
-</xacro:rgbd_sensor_depth_macro>
+    namespace="${namespace}" parent_link="${namespace}/base_link"
+    camera_suffix="depth"
+    frame_rate="30.0"
+    fov = "1.59174"
+    baseline = "0.05"
+    width = "848"
+    height = "480"
+    max_range="50.0"
+    min_range="0.195">
+    <origin xyz="0.2 0.0 -0.05" rpy="0 0.1 0" />
+  </xacro:rgbd_sensor_depth_macro>
 </robot>
